File: KiCad/KiCad.kicad_sch (KiCad schematic)
At the start: 59 parts, among them IC1 LM75AIM_NOPB, J1 Screw_Terminal_01x03, J2 Screw_Terminal_01x03, J3 Screw_Terminal_01x03, J4 Screw_Terminal_01x02, J5 Screw_Terminal_01x02, J6 Screw_Terminal_01x03, J7 Screw_Terminal_01x02, J8 Screw_Terminal_01x03, J9 Screw_Terminal_01x02, Q1 2N3906, Q2 2N3906, Q3 2N3906, Q4 2N3904, Q5 2N3904, Q6 2N3904, Q7 2N3906, Q8 2N3904, U2 L298HN, U3 L7805, U4 ARDUINO_MKR_WAN_1310

Commit message: imp kicad
Parts:
- added C10, C11, C12, C13, C14, C5, C6, C7, C8, C9: 0.1u, Capacitor_SMD:C_1206_3216Metric_Pad1.33x1.80mm_HandSolder, symbol Device:C
- added D13, D14, D15, D16, D17, D18, D19, D20, D21, D22, D23, D24, D25, D26, D27, D28, D29, D30, D31, D32, D33, D34, D35, D36, D37, D38, D39, D40: 1N4007, Diode_SMD:D_1206_3216Metric_Pad1.42x1.75mm_HandSolder, symbol Diode:1N4007
- added D41, D42: 1N5711UR, Diode_SMD:D_1206_3216Metric_Pad1.42x1.75mm_HandSolder, symbol Diode:1N5711UR
- added J10, J11, J12, J13, J14, J15, J16: Screw_Terminal_01x02, TerminalBlock_Phoenix:TerminalBlock_Phoenix_MKDS-1,5-2_1x02_P5.00mm_Horizontal, symbol Connector:Screw_Terminal_01x02
- added J18: Screw_Terminal_01x04, symbol Connector:Screw_Terminal_01x04
- added Q10: 2N3904, Package_TO_SOT_SMD:SOT-23, symbol Transistor_BJT:2N3904
- added Q9: 2N3906, Package_TO_SOT_SMD:SOT-23, symbol Transistor_BJT:2N3906
- added R23: 1.7k, Resistor_SMD:R_1206_3216Metric_Pad1.30x1.75mm_HandSolder, symbol Device:R
- added R24: 3.3k, Resistor_SMD:R_1206_3216Metric_Pad1.30x1.75mm_HandSolder, symbol Device:R
- added R25: 4.7k, Resistor_SMD:R_1206_3216Metric_Pad1.30x1.75mm_HandSolder, symbol Device:R
- added R26: 10k, Resistor_SMD:R_1206_3216Metric_Pad1.30x1.75mm_HandSolder, symbol Device:R
- added R27: 27k, Resistor_SMD:R_1206_3216Metric_Pad1.30x1.75mm_HandSolder, symbol Device:R
- added U1, U5, U6: L298HN, Package_TO_SOT_THT:TO-220-15_P2.54x2.54mm_StaggerOdd_Lead4.58mm_Vertical, symbol Driver_Motor:L298HN
Connections:
- net S3_EN is gone; now on net S_HUM_1_EN: U4.J3_9 (PA22/D0(PWM))
- net S4_EN is gone; now on net S_ILUM_EN: R22.2
- net S4_IN is gone; now on net S_ILUM_IN: D11.2 (A), D12.1 (K), R18.2, R19.1
- net +12V: now also C10.1, C12.1, C13.1, C5.1, C6.1, C7.1, C9.1, D13.1 (K), D15.1 (K), D17.1 (K), D19.1 (K), D21.1 (K), D23.1 (K), D25.1 (K), D27.1 (K), D29.1 (K), D31.1 (K), D33.1 (K), D35.1 (K), D37.1 (K), D39.1 (K), U1.4 (Vs), U5.4 (Vs), U6.4 (Vs)
- net +3V3: now also D41.1 (K), R26.2
- net +5V: now also C11.1, C14.1, C8.1, J18.1 (Pin_1), Q9.1 (E), U1.9 (Vss), U5.9 (Vss), U6.9 (Vss); no longer J8.1 (Pin_1)
- net Earth: now also U2.1 (SENSE_A), C10.2, C11.2, C12.2, C13.2, C14.2, C5.2, C6.2, C7.2, C8.2, C9.2, D14.2 (A), D16.2 (A), D18.2 (A), D20.2 (A), D22.2 (A), D24.2 (A), D26.2 (A), D28.2 (A), D30.2 (A), D32.2 (A), D34.2 (A), D36.2 (A), D38.2 (A), D40.2 (A), D42.2 (A), J18.4 (Pin_4), Q10.1 (E), R24.2, U1.1 (SENSE_A), U1.15 (SENSE_B), U1.8 (GND), U5.1 (SENSE_A), U5.15 (SENSE_B), U5.8 (GND), U6.1 (SENSE_A), U6.15 (SENSE_B), U6.8 (GND)
- net FOCO_EN: now also U4.J3_14 (PB11/D5(PWM))
- net HEAT_EN: now also U4.J5_1 (PA20/D6(PWM))
- net SCL: now also J18.3 (Pin_3)
- net SDA: now also J18.2 (Pin_2)
- net S_HUM_1_IN: now also U4.J3_2 (PA02/D15/DAC0/AIN(0)/A0)
- net S_HUM_2_EN: now also U4.J3_10 (PA23/D1(PWM))
- net S_HUM_2_IN: now also U4.J3_1 (PA03/AREF/AIN(1))
- net S_HUM_3_EN: now also U4.J3_11 (PA10/D2(PWM))
- net S_HUM_3_IN: now also U4.J3_5 (PA04/D18(PWM)/AIN(4)/A3)
- net S_ILUM_EN: now reaches U4.J3_12 (PA11/D3(PWM))
- net S_ANEM_EN: now reaches U4.J3_13 (PB10/D4(PWM))
- net S_ANEM_EN: now also R27.2
- net S_ILUM_IN: now reaches U4.J3_6 (PA05/D19(PWM)/AIN(5)/A4)
- net S_ANEM_IN: now reaches U4.J3_7 (PA06/D20/AIN(6)/A5)
- net S_ANEM_IN: now also D41.2 (A), D42.1 (K), R23.2, R24.1
- net at U2.2 (OUT1): now also D15.2 (A), D16.1 (K), J10.1 (Pin_1)
- net at U2.3 (OUT2): now also D13.2 (A), D14.1 (K), J10.2 (Pin_2)
- net P1_IN2: now reaches U2.5 (IN1)
- net P1_EN: now reaches U2.6 (EnA)
- net P1_IN1: now reaches U2.7 (IN2)
- net ANEMOM_IN: no longer names the net of J8.2 (Pin_2)
- net ANEMOM_IN: now also R23.1
- net D1_IN renamed P2_IN1
- net D2_IN renamed P2_IN2
- net D_EN renamed P2_EN
- new net: D19.2 (A), D20.1 (K), J11.1 (Pin_1), U1.13 (OUT3)
- new net: D39.2 (A), D40.1 (K), J16.1 (Pin_1), U6.2 (OUT1)
- new net: D37.2 (A), D38.1 (K), J16.2 (Pin_2), U6.3 (OUT2)
- new net: D25.2 (A), D26.1 (K), J13.2 (Pin_2), U5.14 (OUT4)
- new net: D27.2 (A), D28.1 (K), J13.1 (Pin_1), U5.13 (OUT3)
- new net: D35.2 (A), D36.1 (K), J15.1 (Pin_1), U6.13 (OUT3)
- new net: Q9.2 (B), R25.2
- new net: J8.1 (Pin_1), Q9.3 (C)
- new net: D17.2 (A), D18.1 (K), J11.2 (Pin_2), U1.14 (OUT4)
- new net: D31.2 (A), D32.1 (K), J14.1 (Pin_1), U5.2 (OUT1)
- new net: D29.2 (A), D30.1 (K), J14.2 (Pin_2), U5.3 (OUT2)
- new net: Q10.2 (B), R27.1
- new net: D21.2 (A), D22.1 (K), J12.2 (Pin_2), U1.3 (OUT2)
- new net: Q10.3 (C), R25.1, R26.1
- new net: D23.2 (A), D24.1 (K), J12.1 (Pin_1), U1.2 (OUT1)
- new net: D33.2 (A), D34.1 (K), J15.2 (Pin_2), U6.14 (OUT4)
- new net P3_EN: U1.6 (EnA)
- new net P3_IN1: U1.7 (IN2)
- new net P3_IN2: U1.5 (IN1)
- new net P4_EN: U1.11 (EnB)
- new net P4_IN1: U1.12 (IN4)
- new net P4_IN2: U1.10 (IN3)
- new net P5_EN: U5.6 (EnA)
- new net P5_IN1: U5.7 (IN2)
- new net P5_IN2: U5.5 (IN1)
- new net W1_EN: U5.11 (EnB)
- new net W1_IN1: U5.12 (IN4)
- new net W1_IN2: U5.10 (IN3)
- new net W2_EN: U6.6 (EnA)
- new net W2_IN1: U6.7 (IN2)
- new net W2_IN2: U6.5 (IN1)
- no-connect marks 8 -> 5
Other:
- note added: "Pump 1"
- note added: "Pump 2"
- note added: "Pump 3"
- note added: "Pump 4"
- note added: "Pump 5"
- note added: "Sensor cond."
- note added: "Window 1"
- note added: "Window 2"
- note removed: "Pump Driver"
- moved on the sheet: D1, D10, D11, D12, D2, D3, D4, D5, D6, D7, D8, D9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
