File: KiCad/KiCad.kicad_sch (KiCad schematic)
At the start: 117 parts, among them IC1 LM75AIM_NOPB, J1 Screw_Terminal_01x03, J10 Screw_Terminal_01x02, J11 Screw_Terminal_01x02, J12 Screw_Terminal_01x02, J13 Screw_Terminal_01x02, J14 Screw_Terminal_01x02, J15 Screw_Terminal_01x02, J16 Screw_Terminal_01x02, J18 Screw_Terminal_01x04, J2 Screw_Terminal_01x03, J3 Screw_Terminal_01x03, J4 Screw_Terminal_01x02, J5 Screw_Terminal_01x02, J6 Screw_Terminal_01x03, J7 Screw_Terminal_01x02, J8 Screw_Terminal_01x03, J9 Screw_Terminal_01x02, Q1 2N3906, Q10 2N3904, Q2 2N3906, Q3 2N3906, Q4 2N3904, Q5 2N3904, Q6 2N3904, Q7 2N3906, Q8 2N3904, Q9 2N3906, U1 L298HN, U2 L298HN, U3 L7805, U4 ARDUINO_MKR_WAN_1310, U5 L298HN, U6 L298HN

Commit message: more kicad
Parts:
- added U8: MAX7300, symbol SamacSys_Parts:MAX7300
Connections:
- no-connect marks 5 -> 7
Changed lines of the file:
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@@
   )
   (no_connect (at 176.53 33.02))
+  (no_connect (at 242.57 60.96))
+  (no_connect (at 242.57 58.42))
   (no_connect (at 168.91 165.1))
   (no_connect (at 370.84 71.12))
@@
     (stroke (width 0) (type default))
   )
-  (wire (pts (xy 378.46 163.83) (xy 378.46 170.18))
+  (wire (pts (xy 378.46 165.1) (xy 378.46 170.18))
     (stroke (width 0) (type default))
   )
@@
     (stroke (width 0) (type default))
   )
-  (wire (pts (xy 375.92 163.83) (xy 375.92 170.18))
+  (wire (pts (xy 375.92 165.1) (xy 375.92 170.18))
     (stroke (width 0) (type default))
   )
@@
     (stroke (width 0) (type default))
   )
-  (wire (pts (xy 381 163.83) (xy 381 170.18))
+  (wire (pts (xy 381 165.1) (xy 381 170.18))
     (stroke (width 0) (type default))
   )
@@
     (effects (font (size 1.27 1.27) bold) (justify left top))
   )
-  (text_box "NOT?"
-    (at 368.3 147.32 0) (size 16.51 6.35)
+  (text_box "21 puertos\n7 libres en ard"
+    (at 313.69 62.23 0) (size 20.32 8.89)
     (stroke (width 0) (type default))
     (fill (type none))
@@
     (effects (font (size 1.27 1.27) (thickness 0.254) bold) (justify left bottom))
   )
+  (label "P3_EN" (at 300.99 85.09 180) (fields_autoplaced)
+    (effects (font (size 1.27 1.27)) (justify right bottom))
+  )
+  (label "P4_EN" (at 300.99 95.25 180) (fields_autoplaced)
+    (effects (font (size 1.27 1.27)) (justify right bottom))
+  )
+  (label "P2_IN2" (at 300.99 67.31 180) (fields_autoplaced)
+    (effects (font (size 1.27 1.27)) (justify right bottom))
+  )
   (label "P3_IN2" (at 316.23 165.1 90) (fields_autoplaced)
     (effects (font (size 1.27 1.27)) (justify left bottom))
@@
     (effects (font (size 1.27 1.27)) (justify left bottom))
   )
+  (label "P4_IN1" (at 300.99 92.71 180) (fields_autoplaced)
+    (effects (font (size 1.27 1.27)) (justify right bottom))
+  )
+  (label "P5_EN" (at 300.99 109.22 180) (fields_autoplaced)
+    (effects (font (size 1.27 1.27)) (justify right bottom))
+  )
+  (label "W2_IN1" (at 300.99 129.54 180) (fields_autoplaced)
+    (effects (font (size 1.27 1.27)) (justify right bottom))
+  )
   (label "P5_IN1" (at 247.65 165.1 90) (fields_autoplaced)
     (effects (font (size 1.27 1.27)) (justify left bottom))
@@
     (effects (font (size 1.27 1.27)) (justify left bottom))
   )
-  (label "P1_IN2" (at 381 163.83 90) (fields_autoplaced)
+  (label "P1_IN2" (at 381 165.1 90) (fields_autoplaced)
     (effects (font (size 1.27 1.27)) (justify left bottom))
   )
@@
     (effects (font (size 1.27 1.27)) (justify left bottom))
   )
+  (label "P1_IN2" (at 299.72 57.15 180) (fields_autoplaced)
+    (effects (font (size 1.27 1.27)) (justify right bottom))
+  )
   (label "W1_EN" (at 234.95 165.1 90) (fields_autoplaced)
     (effects (font (size 1.27 1.27)) (justify left bottom))
@@
     (effects (font (size 1.27 1.27)) (justify left bottom))
   )
+  (label "W2_IN2" (at 300.99 127 180) (fields_autoplaced)
+    (effects (font (size 1.27 1.27)) (justify right bottom))
+  )
+  (label "P1_EN" (at 299.72 62.23 180) (fields_autoplaced)
+    (effects (font (size 1.27 1.27)) (justify right bottom))
+  )
   (label "S_HUM_3_EN" (at 161.29 58.42 0) (fields_autoplaced)
     (effects (font (size 1.27 1.27)) (justify left bottom))
@@
     (effects (font (size 1.27 1.27)) (justify left bottom))
   )
+  (label "W1_EN" (at 300.99 119.38 180) (fields_autoplaced)
+    (effects (font (size 1.27 1.27)) (justify right bottom))
+  )
   (label "SCL" (at 388.62 91.44 0) (fields_autoplaced)
     (effects (font (size 1.27 1.27)) (justify left bottom))
@@
     (effects (font (size 1.27 1.27)) (justify left bottom))
   )
+  (label "W1_IN2" (at 300.99 114.3 180) (fields_autoplaced)
+    (effects (font (size 1.27 1.27)) (justify right bottom))
+  )
+  (label "P3_IN2" (at 300.99 80.01 180) (fields_autoplaced)
+    (effects (font (size 1.27 1.27)) (justify right bottom))
+  )
+  (label "P5_IN2" (at 300.99 104.14 180) (fields_autoplaced)
+    (effects (font (size 1.27 1.27)) (justify right bottom))
+  )
   (label "S_HUM_1_EN" (at 77.47 38.1 0) (fields_autoplaced)
     (effects (font (size 1.27 1.27)) (justify left bottom))
@@
     (effects (font (size 1.27 1.27)) (justify left bottom))
   )
-  (label "P1_EN" (at 375.92 163.83 90) (fields_autoplaced)
-    (effects (font (size 1.27 1.27)) (justify left bottom))
-  )
-  (label "P1_IN1" (at 378.46 163.83 90) (fields_autoplaced)
+  (label "P1_EN" (at 375.92 165.1 90) (fields_autoplaced)
+    (effects (font (size 1.27 1.27)) (justify left bottom))
+  )
+  (label "P1_IN1" (at 378.46 165.1 90) (fields_autoplaced)
     (effects (font (size 1.27 1.27)) (justify left bottom))
   )
@@
     (effects (font (size 1.27 1.27)) (justify left bottom))
   )
+  (label "W2_EN" (at 300.99 132.08 180) (fields_autoplaced)
+    (effects (font (size 1.27 1.27)) (justify right bottom))
+  )
+  (label "P4_IN2" (at 300.99 90.17 180) (fields_autoplaced)
+    (effects (font (size 1.27 1.27)) (justify right bottom))
+  )
   (label "Vin" (at 384.81 46.99 0) (fields_autoplaced)
     (effects (font (size 1.27 1.27)) (justify left bottom))
@@
     (effects (font (size 1.27 1.27)) (justify left bottom))
   )
+  (label "P2_EN" (at 300.99 72.39 180) (fields_autoplaced)
+    (effects (font (size 1.27 1.27)) (justify right bottom))
+  )
+  (label "P2_IN1" (at 300.99 69.85 180) (fields_autoplaced)
+    (effects (font (size 1.27 1.27)) (justify right bottom))
+  )
   (label "W2_EN" (at 179.07 165.1 90) (fields_autoplaced)
     (effects (font (size 1.27 1.27)) (justify left bottom))
   )
+  (label "P1_IN1" (at 299.72 59.69 180) (fields_autoplaced)
+    (effects (font (size 1.27 1.27)) (justify right bottom))
+  )
+  (label "P5_IN1" (at 300.99 106.68 180) (fields_autoplaced)
+    (effects (font (size 1.27 1.27)) (justify right bottom))
+  )
   (label "P3_IN1" (at 313.69 165.1 90) (fields_autoplaced)
     (effects (font (size 1.27 1.27)) (justify left bottom))
@@
     (effects (font (size 1.27 1.27)) (justify left bottom))
   )
+  (label "W1_IN1" (at 300.99 116.84 180) (fields_autoplaced)
+    (effects (font (size 1.27 1.27)) (justify right bottom))
+  )
   (label "P5_IN2" (at 250.19 165.1 90) (fields_autoplaced)
     (effects (font (size 1.27 1.27)) (justify left bottom))
@@
   (label "S_ILUM_EN" (at 78.74 201.93 0) (fields_autoplaced)
     (effects (font (size 1.27 1.27)) (justify left bottom))
+  )
+  (label "P3_IN1" (at 300.99 82.55 180) (fields_autoplaced)
+    (effects (font (size 1.27 1.27)) (justify right bottom))
   )
   (label "S_ILUM_IN" (at 161.29 45.72 0) (fields_autoplaced)
@@
         )
       )
+    )
+  )
+  (symbol (lib_name "MAX7300_1") (lib_id "SamacSys_Parts:MAX7300") (at 381 104.14 0) (unit 1)
+    (in_bom yes) (on_board yes) (dnp no) (fields_autoplaced)
+    (property "Reference" "U8" (at 385.445 100.33 0)
+      (effects (font (size 1.27 1.27)))
+    )
+    (property "Value" "MAX7300" (at 385.445 102.87 0)
+      (effects (font (size 1.27 1.27)))
+    )
+    (property "Footprint" "" (at 381 104.14 0)
+      (effects (font (size 1.27 1.27)) hide)
+    )
+    (property "Datasheet" "https://www.mouser.es/datasheet/2/609/MAX7300-3130962.pdf" (at 387.35 146.05 0)
+      (effects (font (size 1.27 1.27)) hide)
+    )
+    (pin "1")
+    (pin "10")
+    (pin "11")
+    (pin "12")
+    (pin "13")
+    (pin "14")
+    (pin "15")
+    (pin "16")
+    (pin "17")
+    (pin "18")
+    (pin "19")
+    (pin "2")
+    (pin "20")
+    (pin "21")
+    (pin "22")
+    (pin "23")
+    (pin "24")
+    (pin "25")
+    (pin "26")
+    (pin "27")
+    (pin "28")
+    (pin "3")
+    (pin "4")
+    (pin "5")
+    (pin "6")
+    (pin "7")
+    (pin "8")
+    (pin "9")
+    (instances
+      (project "KiCad"
+        (path "/557850ac-a946-4dff-8187-8978353577df"
+          (reference "U8") (unit 1)
+        )
+      )

Commit message: q
Parts:
- removed U8: MAX7300, symbol SamacSys_Parts:MAX7300
- added C15: 0.47u, Capacitor_SMD:C_1206_3216Metric_Pad1.33x1.80mm_HandSolder, symbol Device:C
- added IC2: MAX7300AAI+, SOP65P778X199-28N, symbol SamacSys_Parts:MAX7300AAI+
- added R28: 39k, Resistor_SMD:R_1206_3216Metric_Pad1.30x1.75mm_HandSolder, symbol Device:R
Connections:
- net +3.3V: now also C15.1, IC2.28 (V+)
- net Earth: now also C15.2, IC2.2 (GND_1), IC2.27 (AD1), IC2.3 (GND_2), IC2.4 (AD0), R28.2
- net P1_EN: now also IC2.7 (P14)
- net P1_IN1: now also IC2.6 (P13)
- net P1_IN2: now also IC2.5 (P12)
- net P2_EN: now also IC2.10 (P17)
- net P2_IN1: now also IC2.9 (P16)
- net P2_IN2: now also IC2.8 (P15)
- net P3_EN: now also IC2.13 (P20)
- net P3_IN1: now also IC2.12 (P19)
- net P3_IN2: now also IC2.11 (P18)
- net P4_EN: now also IC2.21 (P28)
- net P4_IN1: now also IC2.22 (P29)
- net P4_IN2: now also IC2.23 (P30)
- net P5_EN: now also IC2.18 (P25)
- net P5_IN1: now also IC2.19 (P26)
- net P5_IN2: now also IC2.20 (P27)
- net SCL: now also IC2.25 (SDA)
- net SDA: now also IC2.26 (SCL)
- net W1_EN: now also IC2.15 (P22)
- net W1_IN1: now also IC2.16 (P23)
- net W1_IN2: now also IC2.17 (P24)
- new net: IC2.1 (ISET), R28.1

Commit message: q
Parts:
- removed C15: 0.47u, Capacitor_SMD:C_1206_3216Metric_Pad1.33x1.80mm_HandSolder, symbol Device:C
- removed IC1: LM75AIM_NOPB, SOIC127P600X175-8N, symbol SamacSys_Parts:LM75AIM_NOPB
- removed IC2: MAX7300AAI+, SOP65P778X199-28N, symbol SamacSys_Parts:MAX7300AAI+
- removed R28: 39k, Resistor_SMD:R_1206_3216Metric_Pad1.30x1.75mm_HandSolder, symbol Device:R
- added IC2, IC3: MCP23017-E_SO, SamacSys_Parts:SOIC127P1030X265-28N, symbol SamacSys_Parts:MCP23017-E_SO
- added U7: LM75AIMX_NOPB, SamacSys_Parts:SOIC127P600X175-8N, symbol SamacSys_Parts:LM75AIMX_NOPB
- J1, J2, J3, J6, J8: footprint (none) -> TerminalBlock_Phoenix:TerminalBlock_Phoenix_MKDS-1,5-3_1x03_P5.00mm_Horizontal
- J18: footprint (none) -> TerminalBlock_Phoenix:TerminalBlock_Phoenix_MKDS-1,5-4_1x04_P5.00mm_Horizontal
- J7, J9: footprint (none) -> TerminalBlock_Phoenix:TerminalBlock_Phoenix_MKDS-1,5-2_1x02_P5.00mm_Horizontal
- R16: value 4.7k -> PAD
- R17: value R -> PAD
Connections:
- net +3.3V: now also IC2.9 (VDD), IC3.9 (VDD)
- net +5V: now also U7.8 (+VS)
- net Earth: now also IC2.10 (VSS), IC2.15 (A0), IC2.16 (A1), IC2.17 (A2), IC3.10 (VSS), IC3.15 (A0), IC3.16 (A1), IC3.17 (A2), U7.4 (GND), U7.5 (A2), U7.6 (A1), U7.7 (A0)
- net P1_EN: now also IC3.1 (GPB0)
- net P1_IN1: now also IC3.2 (GPB1)
- net P1_IN2: now also IC3.3 (GPB2)
- net P2_EN: now also IC3.4 (GPB3)
- net P2_IN1: now also IC3.5 (GPB4)
- net P2_IN2: now also IC3.6 (GPB5)
- net P3_EN: now also IC3.7 (GPB6)
- net P3_IN1: now also IC3.8 (GPB7)
- net P3_IN2: now also IC3.21 (GPA0)
- net P4_EN: now also IC3.22 (GPA1)
- net P4_IN1: now also IC3.23 (GPA2)
- net P4_IN2: now also IC3.24 (GPA3)
- net P5_EN: now also IC3.25 (GPA4)
- net P5_IN1: now also IC3.26 (GPA5)
- net P5_IN2: now also IC3.27 (GPA6)
- net SCL: now also IC2.13 (SDA), IC3.13 (SDA), U7.2 (SCL)
- net SDA: now also IC2.12 (SCL), IC3.12 (SCL), U7.1 (SDA)
- net W1_EN: now also IC2.21 (GPA0)
- net W1_IN1: now also IC2.22 (GPA1)
- net W1_IN2: now also IC2.23 (GPA2)
- net W2_EN: now also IC2.24 (GPA3)
- net W2_IN1: now also IC2.25 (GPA4)
- net W2_IN2: now also IC2.26 (GPA5)
- net R1_IN2: now reaches U6.10 (IN3)
- net R1_IN2: now also IC2.3 (GPB2)
- net R1_EN: now reaches U6.11 (EnB)
- net R1_EN: now also IC2.1 (GPB0)
- net R1_IN1: now reaches U6.12 (IN4)
- net R1_IN1: now also IC2.2 (GPB1)
- no-connect marks 7 -> 29
Other:
- note added: "Port expansion for motor"
- note added: "Reserve 1"
- moved on the sheet: D10, D13, D14, D15, D16, D17, D18, D19, D20, D21, D22, D23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
