File: KiCad/KiCad.kicad_sch (KiCad schematic)
At the start: 130 parts, among them IC1 MCP23017-E_SO, IC2 MCP23017-E_SO, J1 Screw_Terminal_01x03, J10 Screw_Terminal_01x05, J11 Screw_Terminal_01x02, J12 Screw_Terminal_01x02, J13 Screw_Terminal_01x04, J14 Screw_Terminal_01x02, J15 Screw_Terminal_01x02, J16 Screw_Terminal_01x02, J17 Screw_Terminal_01x02, J18 Screw_Terminal_01x02, J19 Screw_Terminal_01x02, J2 Screw_Terminal_01x03, J3 Screw_Terminal_01x03, J4 Screw_Terminal_01x03, J5 Screw_Terminal_01x03, J6 Screw_Terminal_01x02, J7 Screw_Terminal_01x02, J8 Screw_Terminal_01x02, J9 Screw_Terminal_01x02, K1 2071556-9, K2 2071556-9, Q1 2N3906, Q10 2N3904, Q11 2N3904, Q12 2N3904, Q2 2N3906, Q3 2N3906, Q4 2N3906, Q5 2N3906, Q6 2N3904, Q7 2N3904, Q8 2N3904, Q9 2N3904, SW1 SW_Push, U1 L298HN, U2 ARDUINO_MKR_WAN_1310, U3 L298HN, U4 L298HN, U5 L298HN, U6 LM75AIMX_NOPB, U7 L7805

Commit message: sch cahnges
Parts:
- removed C15: 0.1u, Capacitor_SMD:C_1206_3216Metric_Pad1.33x1.80mm_HandSolder, symbol Device:C
- removed D10, D9: 1N5711UR, Diode_SMD:D_1206_3216Metric_Pad1.42x1.75mm_HandSolder, symbol Diode:1N5711UR
- removed Q10: 2N3904, Package_TO_SOT_SMD:SOT-23, symbol Transistor_BJT:2N3904
- removed Q5: 2N3906, Package_TO_SOT_SMD:SOT-23, symbol Transistor_BJT:2N3906
- removed R10: 3.3k, Resistor_SMD:R_1206_3216Metric_Pad1.30x1.75mm_HandSolder, symbol Device:R
- removed R15: 4.7k, Resistor_SMD:R_1206_3216Metric_Pad1.30x1.75mm_HandSolder, symbol Device:R
- removed R20: 10k, Resistor_SMD:R_1206_3216Metric_Pad1.30x1.75mm_HandSolder, symbol Device:R
- removed R25: 27k, Resistor_SMD:R_1206_3216Metric_Pad1.30x1.75mm_HandSolder, symbol Device:R
- removed R9: 1.7k, Resistor_SMD:R_1206_3216Metric_Pad1.30x1.75mm_HandSolder, symbol Device:R
- removed U6: LM75AIMX_NOPB, SamacSys_Parts:SOIC127P600X175-8N, symbol SamacSys_Parts:LM75AIMX_NOPB
- added IC3: DS89C21TMX_NOPB, SOIC127P600X175-8N, symbol SamacSys_Parts:DS89C21TMX_NOPB
- added J20: Screw_Terminal_01x05, TerminalBlock_Phoenix:TerminalBlock_Phoenix_MKDS-1,5-5_1x05_P5.00mm_Horizontal, symbol Connector:Screw_Terminal_01x05
Connections:
- net +5V: now also IC3.1 (VCC)
- net Earth: now also IC3.4 (GND), J20.5 (Pin_5)
- net S_ANEM_IN: now also J5.2 (Pin_2)
- net +9V: now reaches J5.1 (Pin_1)
- net RX: now reaches U2.J5_8 (PB23/D13/RX(SC5))
- net RX: now also IC3.2 (RO)
- net TX: now reaches U2.J5_9 (PB22/D14/TX(SC5))
- net TX: now also IC3.3 (DI)
- net S_ANEM_EN: no longer names the net of U2.J3_13 (PB10/D4(PWM))
- new net D0_1: IC3.5 (DO_1), J20.1 (Pin_1)
- new net D0_2: IC3.6 (DO_2), J20.2 (Pin_2)
- new net RI_1: IC3.7 (RI_1), J20.3 (Pin_3)
- new net RI_2: IC3.8 (RI_2), J20.4 (Pin_4)
- no-connect marks 23 -> 21
Other:
- note added: "RS422"
- note removed: "Temp. Sensor"
