File: KiCad/SalveNode/SalveNode.kicad_sch (KiCad schematic)
At the start: 2 parts, among them IC1 TMP75AQDGKRQ1

Commit message: tarjeta externa añadido
Parts:
- removed A1: Arduino_UNO_R2, Module:Arduino_UNO_R2, symbol MCU_Module:Arduino_UNO_R2
- added A1: ALS-PT19-315C_L177_TR8, ALS-PT19-315C_L177_TR8:XDCR_ALS-PT19-315C_L177_TR8, symbol ALS-PT19-315C_L177_TR8:ALS-PT19-315C_L177_TR8
- added IC3: ATMEGA328PB-AN, QFP80P900X900X120-32N, symbol SamacSys_Parts:ATMEGA328PB-AN
- added IC3: DS89C21TMX_NOPB, SOIC127P600X175-8N, symbol SamacSys_Parts:DS89C21TMX_NOPB
- added J1, J21: Screw_Terminal_01x06, symbol Connector:Screw_Terminal_01x06
- added R1: 10k, symbol Device:R
- added R7: PAD, Resistor_SMD:R_1206_3216Metric_Pad1.30x1.75mm_HandSolder, symbol Device:R
- renumbered IC1 to IC2
Connections:
- net +5V: now also A1.1, IC3.1 (VCC), IC3.18 (AVCC), IC3.4 (VCC), J1.1 (Pin_1), J21.1 (Pin_1), R1.2
- net Earth: now also IC3.20 (AREF), IC3.21 (GND_2), IC3.4 (GND), IC3.5 (GND_1), J1.6 (Pin_6), J21.6 (Pin_6)
- net RX: now also IC3.2 (RO), IC3.30 (PD0_(PTCXY/OC3A/RXD0))
- net SCL: now also IC3.28 (PC5_(ADC5/PTCY/SCL0))
- net SDA: now also IC3.27 (PC4_(ADC4/PTCY/SDA0))
- net TX: now also IC3.3 (DI), IC3.31 (PD1_(PTCXY/OC4A/TXD0))
- new net D0_1: IC3.5 (DO_1), J21.2 (Pin_2)
- new net D0_2: IC3.6 (DO_2), J21.3 (Pin_3)
- new net LIGHT_IN: A1.2, IC3.23 (PC0_(ADC0/PTCY/MISO1)), R1.1
- new net MISO: IC3.16 ((MISO0/RXD1/PTCXY)_PB4), J1.3 (Pin_3)
- new net MOSI: IC3.15 ((MOSI0/TXD1/OC2A/PTCXY)_PB3), J1.2 (Pin_2)
- new net RESET: IC3.29 (PC6_(~{RESET)}), J1.4 (Pin_4)
- new net RI_1: IC3.7 (RI_1), J21.4 (Pin_4), R7.2
- new net RI_2: IC3.8 (RI_2), J21.5 (Pin_5), R7.1
- new net SCK: IC3.17 (PB5_(PTCXY/XCK1/SCK0)), J1.5 (Pin_5)
- no-connect marks 5 -> 19
Other:
- note added: "Light"
- note added: "Power and serial"
- note added: "Programming"
- note added: "RS422"
- note added: "Temperature"
- moved on the sheet: IC2

Commit message: sch complete
Parts:
- added C1, C2: C, Capacitor_SMD:C_1206_3216Metric_Pad1.33x1.80mm_HandSolder, symbol Device:C
- added Y2: Crystal, Crystal:Crystal_HC18-U_Vertical, symbol Device:Crystal
- A1: footprint ALS-PT19-315C_L177_TR8:XDCR_ALS-PT19-315C_L177_TR8 -> SimbolosSnapEDA:XDCR_ALS-PT19-315C_L177_TR8
- IC2: footprint SOP65P490X110-8N -> SamacSys_Parts:SOP65P490X110-8N
- IC3: footprint QFP80P900X900X120-32N -> SamacSys_Parts:QFP80P900X900X120-32N
- IC3: footprint SOIC127P600X175-8N -> SamacSys_Parts:SOIC127P600X175-8N
- J1, J21: footprint (none) -> TerminalBlock_Phoenix:TerminalBlock_Phoenix_MKDS-1,5-6_1x06_P5.00mm_Horizontal
- R1: footprint (none) -> Resistor_SMD:R_1206_3216Metric_Pad1.30x1.75mm_HandSolder
Connections:
- net Earth: now also C1.1, C2.1
- net XTAL1: now reaches IC3.7 ((XTAL1/TOSC1)_PB6)
- net XTAL1: now also C1.2, Y2.2
- net XTAL2: now reaches IC3.8 ((XTAL2/TOSC2)_PB7)
- net XTAL2: now also C2.2, Y2.1
- no-connect marks 19 -> 17
Changed lines of the file:
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@@
 (kicad_sch (version 20230121) (generator eeschema)
   (paper "A4")
+  (junction (at 97.79 24.13) (diameter 0) (color 0 0 0 0)
+  )
   (junction (at 34.29 29.21) (diameter 0) (color 0 0 0 0)
   )
@@
   (junction (at 54.61 116.84) (diameter 0) (color 0 0 0 0)
   )
+  (junction (at 105.41 35.56) (diameter 0) (color 0 0 0 0)
+  )
+  (junction (at 111.76 24.13) (diameter 0) (color 0 0 0 0)
+  )
   (junction (at 21.59 29.21) (diameter 0) (color 0 0 0 0)
   )
@@
   )
   (no_connect (at 231.14 96.52))
-  (no_connect (at 182.88 137.16))
   (no_connect (at 167.64 137.16))
   (no_connect (at 180.34 137.16))
@@
   (no_connect (at 231.14 99.06))
   (no_connect (at 170.18 137.16))
-  (no_connect (at 185.42 137.16))
   (no_connect (at 167.64 55.88))
   (no_connect (at 124.46 88.9))
@@
     (stroke (width 0) (type default))
   )
+  (wire (pts (xy 109.22 24.13) (xy 111.76 24.13))
+    (stroke (width 0) (type default))
+  )
   (wire (pts (xy 58.42 57.15) (xy 58.42 59.69))
     (stroke (width 0) (type default))
@@
     (stroke (width 0) (type default))
   )
+  (wire (pts (xy 97.79 35.56) (xy 105.41 35.56))
+    (stroke (width 0) (type default))
+  )
   (wire (pts (xy 24.13 27.94) (xy 24.13 33.02))
     (stroke (width 0) (type default))
@@
     (stroke (width 0) (type default))
   )
+  (wire (pts (xy 111.76 24.13) (xy 119.38 24.13))
+    (stroke (width 0) (type default))
+  )
+  (wire (pts (xy 97.79 27.94) (xy 97.79 24.13))
+    (stroke (width 0) (type default))
+  )
+  (wire (pts (xy 111.76 24.13) (xy 111.76 27.94))
+    (stroke (width 0) (type default))
+  )
+  (wire (pts (xy 105.41 35.56) (xy 111.76 35.56))
+    (stroke (width 0) (type default))
+  )
   (wire (pts (xy 25.4 83.82) (xy 25.4 96.52))
     (stroke (width 0) (type default))
   )
+  (wire (pts (xy 90.17 24.13) (xy 97.79 24.13))
+    (stroke (width 0) (type default))
+  )
+  (wire (pts (xy 185.42 137.16) (xy 185.42 144.78))
+    (stroke (width 0) (type default))
+  )
   (wire (pts (xy 17.78 59.69) (xy 21.59 59.69))
     (stroke (width 0) (type default))
@@
     (stroke (width 0) (type default))
   )
+  (wire (pts (xy 97.79 24.13) (xy 101.6 24.13))
+    (stroke (width 0) (type default))
+  )
+  (wire (pts (xy 182.88 137.16) (xy 182.88 144.78))
+    (stroke (width 0) (type default))
+  )
   (wire (pts (xy 52.07 111.76) (xy 54.61 111.76))
     (stroke (width 0) (type default))
@@
   )
   (wire (pts (xy 24.13 146.05) (xy 24.13 148.59))
+    (stroke (width 0) (type default))
+  )
+  (wire (pts (xy 105.41 35.56) (xy 105.41 36.83))
     (stroke (width 0) (type default))
   )
@@
     (effects (font (size 1.27 1.27)) (justify right bottom))
   )
+  (label "XTAL1" (at 182.88 144.78 90) (fields_autoplaced)
+    (effects (font (size 1.27 1.27)) (justify left bottom))
+  )
   (label "RX" (at 118.11 101.6 0) (fields_autoplaced)
     (effects (font (size 1.27 1.27)) (justify left bottom))
@@
     (effects (font (size 1.27 1.27)) (justify left bottom))
   )
+  (label "XTAL2" (at 185.42 144.78 90) (fields_autoplaced)
+    (effects (font (size 1.27 1.27)) (justify left bottom))
+  )
   (label "D0_1" (at 24.13 33.02 90) (fields_autoplaced)
     (effects (font (size 1.27 1.27)) (justify left bottom))
@@
     (effects (font (size 1.27 1.27)) (justify left bottom))
   )
+  (label "XTAL2" (at 90.17 24.13 0) (fields_autoplaced)
+    (effects (font (size 1.27 1.27)) (justify left bottom))
+  )
   (label "MOSI" (at 22.86 96.52 90) (fields_autoplaced)
     (effects (font (size 1.27 1.27)) (justify left bottom))
   )
   (label "SCK" (at 185.42 44.45 270) (fields_autoplaced)
+    (effects (font (size 1.27 1.27)) (justify right bottom))
+  )
+  (label "XTAL1" (at 119.38 24.13 180) (fields_autoplaced)
     (effects (font (size 1.27 1.27)) (justify right bottom))
   )
@@
       (effects (font (size 1.27 1.27)) (justify left))
     )
-    (property "Footprint" "" (at 22.352 152.4 90)
+    (property "Footprint" "Resistor_SMD:R_1206_3216Metric_Pad1.30x1.75mm_HandSolder" (at 22.352 152.4 90)
       (effects (font (size 1.27 1.27)) hide)
     )
@@
         (path "/947c7390-073c-40c7-ae18-83309c4a488f"
           (reference "R1") (unit 1)
+        )
+      )
+    )
+  )
+  (symbol (lib_id "Device:Crystal") (at 105.41 24.13 0) (unit 1)
+    (in_bom yes) (on_board yes) (dnp no) (fields_autoplaced)
+    (property "Reference" "Y2" (at 105.41 16.51 0)
+      (effects (font (size 1.27 1.27)))
+    )
+    (property "Value" "Crystal" (at 105.41 19.05 0)
+      (effects (font (size 1.27 1.27)))
+    )
+    (property "Footprint" "Crystal:Crystal_HC18-U_Vertical" (at 105.41 24.13 0)
+      (effects (font (size 1.27 1.27)) hide)
+    )
+    (property "Datasheet" "~" (at 105.41 24.13 0)
+      (effects (font (size 1.27 1.27)) hide)
+    )
+    (pin "1")
+    (pin "2")
+    (instances
+      (project "SalveNode"
+        (path "/947c7390-073c-40c7-ae18-83309c4a488f"
+          (reference "Y2") (unit 1)
         )
       )
@@
     )
   )
+  (symbol (lib_id "power:Earth") (at 105.41 36.83 0) (unit 1)
+    (in_bom yes) (on_board yes) (dnp no) (fields_autoplaced)
+    (property "Reference" "#PWR0122" (at 105.41 43.18 0)
+      (effects (font (size 1.27 1.27)) hide)
+    )
+    (property "Value" "Earth" (at 105.41 40.64 0)
+      (effects (font (size 1.27 1.27)) hide)
+    )
+    (property "Footprint" "" (at 105.41 36.83 0)
+      (effects (font (size 1.27 1.27)) hide)
+    )
+    (property "Datasheet" "~" (at 105.41 36.83 0)
+      (effects (font (size 1.27 1.27)) hide)
+    )
+    (pin "1")
+    (instances
+      (project "KiCad"
+        (path "/557850ac-a946-4dff-8187-8978353577df"
+          (reference "#PWR0122") (unit 1)
+        )
+      )
+      (project "SalveNode"
+        (path "/947c7390-073c-40c7-ae18-83309c4a488f"
+          (reference "#PWR016") (unit 1)
+        )
+      )
+    )
+  )
   (symbol (lib_id "ALS-PT19-315C_L177_TR8:ALS-PT19-315C_L177_TR8") (at 21.59 137.16 0) (unit 1)
     (in_bom yes) (on_board yes) (dnp no) (fields_autoplaced)
@@
       (effects (font (size 1.27 1.27)) (justify left))
     )
-    (property "Footprint" "ALS-PT19-315C_L177_TR8:XDCR_ALS-PT19-315C_L177_TR8" (at 21.59 137.16 0)
+    (property "Footprint" "SimbolosSnapEDA:XDCR_ALS-PT19-315C_L177_TR8" (at 21.59 137.16 0)
       (effects (font (size 1.27 1.27)) (justify bottom) hide)
     )
@@
       (effects (font (size 1.27 1.27)))
     )
-    (property "Footprint" "SOP65P490X110-8N" (at 48.26 204.14 0)
+    (property "Footprint" "SamacSys_Parts:SOP65P490X110-8N" (at 48.26 204.14 0)
       (effects (font (size 1.27 1.27)) (justify left top) hide)
     )
@@
       (effects (font (size 1.27 1.27)))
     )
-    (property "Footprint" "QFP80P900X900X120-32N" (at 227 59.69 0)
+    (property "Footprint" "SamacSys_Parts:QFP80P900X900X120-32N" (at 227 59.69 0)
       (effects (font (size 1.27 1.27)) (justify left top) hide)
     )
@@
     )
   )
+  (symbol (lib_id "Device:C") (at 111.76 31.75 180) (unit 1)
+    (in_bom yes) (on_board yes) (dnp no) (fields_autoplaced)
+    (property "Reference" "C1" (at 115.57 30.48 0)
+      (effects (font (size 1.27 1.27)) (justify right))
+    )
+    (property "Value" "C" (at 115.57 33.02 0)
+      (effects (font (size 1.27 1.27)) (justify right))
+    )
+    (property "Footprint" "Capacitor_SMD:C_1206_3216Metric_Pad1.33x1.80mm_HandSolder" (at 110.7948 27.94 0)
+      (effects (font (size 1.27 1.27)) hide)
+    )
+    (property "Datasheet" "~" (at 111.76 31.75 0)
+      (effects (font (size 1.27 1.27)) hide)
+    )
+    (pin "1")
+    (pin "2")
+    (instances
+      (project "SalveNode"
+        (path "/947c7390-073c-40c7-ae18-83309c4a488f"
+          (reference "C1") (unit 1)
+        )
+      )
+    )
+  )
   (symbol (lib_name "Earth_1") (lib_id "power:Earth") (at 33.02 83.82 0) (unit 1)
     (in_bom yes) (on_board yes) (dnp no) (fields_autoplaced)
@@
     )
   )
+  (symbol (lib_id "Device:C") (at 97.79 31.75 180) (unit 1)
+    (in_bom yes) (on_board yes) (dnp no) (fields_autoplaced)
+    (property "Reference" "C2" (at 101.6 30.48 0)
+      (effects (font (size 1.27 1.27)) (justify right))
+    )
+    (property "Value" "C" (at 101.6 33.02 0)
+      (effects (font (size 1.27 1.27)) (justify right))
+    )
+    (property "Footprint" "Capacitor_SMD:C_1206_3216Metric_Pad1.33x1.80mm_HandSolder" (at 96.8248 27.94 0)
+      (effects (font (size 1.27 1.27)) hide)
+    )
+    (property "Datasheet" "~" (at 97.79 31.75 0)
+      (effects (font (size 1.27 1.27)) hide)
+    )
+    (pin "1")
+    (pin "2")
+    (instances
+      (project "SalveNode"
+        (path "/947c7390-073c-40c7-ae18-83309c4a488f"
+          (reference "C2") (unit 1)
+        )
+      )
+    )
+  )
   (symbol (lib_id "Connector:Screw_Terminal_01x06") (at 25.4 78.74 90) (unit 1)
     (in_bom yes) (on_board yes) (dnp no) (fields_autoplaced)
@@
       (effects (font (size 1.27 1.27)))
     )
-    (property "Footprint" "" (at 25.4 78.74 0)
+    (property "Footprint" "TerminalBlock_Phoenix:TerminalBlock_Phoenix_MKDS-1,5-6_1x06_P5.00mm_Horizontal" (at 25.4 78.74 0)
       (effects (font (size 1.27 1.27)) hide)
     )
@@
       (effects (font (size 1.27 1.27)))
     )
-    (property "Footprint" "SOIC127P600X175-8N" (at 45.72 149.53 0)
+    (property "Footprint" "SamacSys_Parts:SOIC127P600X175-8N" (at 45.72 149.53 0)
       (effects (font (size 1.27 1.27)) (justify left top) hide)
     )
@@
       (effects (font (size 1.27 1.27)))
     )
-    (property "Footprint" "" (at 26.67 22.86 0)
-      (effects (font (size 1.27 1.27)) hide)
-    )
+    (property "Footprint" "TerminalBlock_Phoenix:TerminalBlock_Phoenix_MKDS-1,5-6_1x06_P5.00mm_Horizontal" (at 26.67 22.86 0)
+      (effects (font (size 1.27 1.27)) hide)
+    )

Commit message: pcb
Parts:
- renumbered C2 to C1, C1 to C2, Y2 to Y1
Connections:
- net +5V: no longer R1.2
- net Earth: now also R1.2
- net D0_1 renamed D0-
- net D0_2 renamed D0+
- net RI_1 renamed RI-
- net RI_2 renamed RI+
Changed lines of the file:
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@@
     (effects (font (size 1.27 1.27)) (justify left bottom))
   )
-  (label "RI_1" (at 29.21 33.02 90) (fields_autoplaced)
+  (label "RI-" (at 29.21 33.02 90) (fields_autoplaced)
     (effects (font (size 1.27 1.27)) (justify left bottom))
   )
@@
     (effects (font (size 1.27 1.27)) (justify left bottom))
   )
-  (label "RI_2" (at 31.75 33.02 90) (fields_autoplaced)
+  (label "RI+" (at 31.75 33.02 90) (fields_autoplaced)
     (effects (font (size 1.27 1.27)) (justify left bottom))
   )
@@
     (effects (font (size 1.27 1.27)) (justify left bottom))
   )
-  (label "D0_1" (at 24.13 33.02 90) (fields_autoplaced)
+  (label "D0-" (at 24.13 33.02 90) (fields_autoplaced)
     (effects (font (size 1.27 1.27)) (justify left bottom))
   )
@@
     (effects (font (size 1.27 1.27)) (justify left bottom))
   )
-  (label "RI_1" (at 68.58 59.69 0) (fields_autoplaced)
+  (label "RI-" (at 68.58 59.69 0) (fields_autoplaced)
     (effects (font (size 1.27 1.27)) (justify left bottom))
   )
@@
     (effects (font (size 1.27 1.27)) (justify left bottom))
   )
-  (label "RI_2" (at 68.58 52.07 0) (fields_autoplaced)
-    (effects (font (size 1.27 1.27)) (justify left bottom))
-  )
-  (label "D0_2" (at 26.67 33.02 90) (fields_autoplaced)
+  (label "RI+" (at 68.58 52.07 0) (fields_autoplaced)
+    (effects (font (size 1.27 1.27)) (justify left bottom))
+  )
+  (label "D0+" (at 26.67 33.02 90) (fields_autoplaced)
     (effects (font (size 1.27 1.27)) (justify left bottom))
   )
@@
     (effects (font (size 1.27 1.27)) (justify right bottom))
   )
-  (label "D0_2" (at 54.61 59.69 180) (fields_autoplaced)
+  (label "D0+" (at 54.61 59.69 180) (fields_autoplaced)
     (effects (font (size 1.27 1.27)) (justify right bottom))
   )
@@
     (effects (font (size 1.27 1.27)) (justify left bottom))
   )
-  (label "D0_1" (at 54.61 62.23 180) (fields_autoplaced)
+  (label "D0-" (at 54.61 62.23 180) (fields_autoplaced)
     (effects (font (size 1.27 1.27)) (justify right bottom))
   )
@@
       (project "SalveNode"
         (path "/947c7390-073c-40c7-ae18-83309c4a488f"
-          (reference "#PWR013") (unit 1)
+          (reference "#PWR014") (unit 1)
         )
       )
@@
   (symbol (lib_id "Device:Crystal") (at 105.41 24.13 0) (unit 1)
     (in_bom yes) (on_board yes) (dnp no) (fields_autoplaced)
-    (property "Reference" "Y2" (at 105.41 16.51 0)
+    (property "Reference" "Y1" (at 105.41 16.51 0)
       (effects (font (size 1.27 1.27)))
     )
@@
       (project "SalveNode"
         (path "/947c7390-073c-40c7-ae18-83309c4a488f"
-          (reference "Y2") (unit 1)
+          (reference "Y1") (unit 1)
         )
       )
@@
   (symbol (lib_id "power:+5V") (at 175.26 137.16 180) (unit 1)
     (in_bom yes) (on_board yes) (dnp no) (fields_autoplaced)
-    (property "Reference" "#PWR012" (at 175.26 133.35 0)
+    (property "Reference" "#PWR013" (at 175.26 133.35 0)
       (effects (font (size 1.27 1.27)) hide)
     )
@@
       (project "SalveNode"
         (path "/947c7390-073c-40c7-ae18-83309c4a488f"
-          (reference "#PWR012") (unit 1)
+          (reference "#PWR013") (unit 1)
         )
       )
@@
       (project "SalveNode"
         (path "/947c7390-073c-40c7-ae18-83309c4a488f"
-          (reference "#PWR016") (unit 1)
+          (reference "#PWR012") (unit 1)
         )
       )
@@
     )
   )
-  (symbol (lib_id "power:+5V") (at 24.13 156.21 180) (unit 1)
-    (in_bom yes) (on_board yes) (dnp no) (fields_autoplaced)
-    (property "Reference" "#PWR07" (at 24.13 152.4 0)
-      (effects (font (size 1.27 1.27)) hide)
-    )
-    (property "Value" "+5V" (at 24.13 161.29 0)
-      (effects (font (size 1.27 1.27)))
-    )
-    (property "Footprint" "" (at 24.13 156.21 0)
-      (effects (font (size 1.27 1.27)) hide)
-    )
-    (property "Datasheet" "" (at 24.13 156.21 0)
-      (effects (font (size 1.27 1.27)) hide)
-    )
-    (pin "1")
-    (instances
-      (project "SalveNode"
-        (path "/947c7390-073c-40c7-ae18-83309c4a488f"
-          (reference "#PWR07") (unit 1)
-        )
-      )
-    )
-  )
   (symbol (lib_id "Device:R") (at 62.23 55.88 0) (mirror y) (unit 1)
     (in_bom yes) (on_board yes) (dnp no) (fields_autoplaced)
@@
   (symbol (lib_id "Device:C") (at 111.76 31.75 180) (unit 1)
     (in_bom yes) (on_board yes) (dnp no) (fields_autoplaced)
-    (property "Reference" "C1" (at 115.57 30.48 0)
+    (property "Reference" "C2" (at 115.57 30.48 0)
       (effects (font (size 1.27 1.27)) (justify right))
     )
@@
       (project "SalveNode"
         (path "/947c7390-073c-40c7-ae18-83309c4a488f"
-          (reference "C1") (unit 1)
+          (reference "C2") (unit 1)
         )
       )
@@
   (symbol (lib_id "Device:C") (at 97.79 31.75 180) (unit 1)
     (in_bom yes) (on_board yes) (dnp no) (fields_autoplaced)
-    (property "Reference" "C2" (at 101.6 30.48 0)
+    (property "Reference" "C1" (at 101.6 30.48 0)
       (effects (font (size 1.27 1.27)) (justify right))
     )
@@
       (project "SalveNode"
         (path "/947c7390-073c-40c7-ae18-83309c4a488f"
-          (reference "C2") (unit 1)
+          (reference "C1") (unit 1)
         )
       )
@@
   (symbol (lib_id "power:Earth") (at 177.8 137.16 0) (unit 1)
     (in_bom yes) (on_board yes) (dnp no) (fields_autoplaced)
-    (property "Reference" "#PWR014" (at 177.8 143.51 0)
+    (property "Reference" "#PWR015" (at 177.8 143.51 0)
       (effects (font (size 1.27 1.27)) hide)
     )
@@
       (project "SalveNode"
         (path "/947c7390-073c-40c7-ae18-83309c4a488f"
-          (reference "#PWR014") (unit 1)
+          (reference "#PWR015") (unit 1)
+        )
+      )
+    )
+  )
+  (symbol (lib_id "power:Earth") (at 24.13 156.21 0) (unit 1)
+    (in_bom yes) (on_board yes) (dnp no) (fields_autoplaced)
+    (property "Reference" "#PWR07" (at 24.13 162.56 0)
+      (effects (font (size 1.27 1.27)) hide)
+    )
+    (property "Value" "Earth" (at 24.13 160.02 0)
+      (effects (font (size 1.27 1.27)) hide)
+    )
+    (property "Footprint" "" (at 24.13 156.21 0)
+      (effects (font (size 1.27 1.27)) hide)
+    )
+    (property "Datasheet" "~" (at 24.13 156.21 0)
+      (effects (font (size 1.27 1.27)) hide)
+    )
+    (pin "1")
+    (instances
+      (project "SalveNode"
+        (path "/947c7390-073c-40c7-ae18-83309c4a488f"
+          (reference "#PWR07") (unit 1)
         )
       )
@@
   (symbol (lib_id "power:+5V") (at 182.88 55.88 0) (unit 1)
     (in_bom yes) (on_board yes) (dnp no) (fields_autoplaced)
-    (property "Reference" "#PWR015" (at 182.88 59.69 0)
+    (property "Reference" "#PWR016" (at 182.88 59.69 0)
       (effects (font (size 1.27 1.27)) hide)
     )
@@
       (project "SalveNode"
         (path "/947c7390-073c-40c7-ae18-83309c4a488f"
-          (reference "#PWR015") (unit 1)
-        )
-      )
+          (reference "#PWR016") (unit 1)
+        )
+      )

Commit message: pcb changes
Parts:
- removed A1: ALS-PT19-315C_L177_TR8, SimbolosSnapEDA:XDCR_ALS-PT19-315C_L177_TR8, symbol ALS-PT19-315C_L177_TR8:ALS-PT19-315C_L177_TR8
- removed R1: 10k, Resistor_SMD:R_1206_3216Metric_Pad1.30x1.75mm_HandSolder, symbol Device:R
- added C3, C4, C5, C6, C7: 100n, Capacitor_SMD:C_1206_3216Metric_Pad1.33x1.80mm_HandSolder, symbol Device:C
- added IC4: VEML7700-TR, SamacSys_Parts:VEML7700, symbol SamacSys_Parts:VEML7700-TR
- added R26, R27: PAD, Resistor_SMD:R_1206_3216Metric_Pad1.30x1.75mm_HandSolder, symbol Device:R
- added R5, R6: R, symbol Device:R
Connections:
- net +5V: now also J1.6 (Pin_6), C3.2, C4.2, C5.2, C6.2, C7.2, R26.1, R27.2, R5.1; no longer J1.1 (Pin_1)
- net Earth: now also J1.1 (Pin_1), C3.1, C4.1, C5.1, C6.1, C7.1, IC4.3 (GND), R6.2; no longer J1.6 (Pin_6)
- net RESET: now also J1.5 (Pin_5); no longer J1.4 (Pin_4)
- net SCK: now also J1.4 (Pin_4); no longer J1.5 (Pin_5)
- net SCL: now also IC4.1 (SCL), R27.1
- net SDA: now also IC4.4 (SDA), R26.2
- new net: IC4.2 (VDD), R5.2, R6.1

Commit message: PCB Complete
Parts:
- removed IC3: ATMEGA328PB-AN, SamacSys_Parts:QFP80P900X900X120-32N, symbol SamacSys_Parts:ATMEGA328PB-AN
- added U1: ATmega328PB-A, Package_QFP:TQFP-32_7x7mm_P0.8mm, symbol MCU_Microchip_ATmega:ATmega328PB-A
- R1: renamed from R5; footprint (none) -> Resistor_SMD:R_1206_3216Metric_Pad1.30x1.75mm_HandSolder
- R2: renamed from R6; footprint (none) -> Resistor_SMD:R_1206_3216Metric_Pad1.30x1.75mm_HandSolder
- renumbered IC4 to IC3
Connections:
- net +5V: now also IC2.5 (A2), IC2.6 (A1), IC2.7 (A0), U1.18 (AVCC), U1.4 (VCC)
- net Earth: now also U1.20 (AREF), U1.21 (GND), U1.5 (GND); no longer IC2.5 (A2), IC2.6 (A1), IC2.7 (A0)
- net MISO: now also U1.16 (PB4)
- net MOSI: now also U1.15 (PB3)
- net RESET: now also U1.29 (~{RESET}/PC6)
- net RX: now also U1.30 (PD0)
- net SCK: now also U1.17 (PB5)
- net SCL: now also U1.28 (PC5)
- net SDA: now also U1.27 (PC4)
- net TX: now also U1.31 (PD1)
- net XTAL1: now also U1.7 (XTAL1/PB6)
- net XTAL2: now also U1.8 (XTAL2/PB7)
- no-connect marks 17 -> 18
