File: KiCad/SalveNode/SalveNode.kicad_sch (KiCad schematic)
At the start: 21 parts, among them IC2 TMP75AQDGKRQ1, IC3 DS89C21TMX_NOPB, IC3 VEML7700-TR, J1 Screw_Terminal_01x06, J21 Screw_Terminal_01x06, U1 ATmega328PB-A, Y1 Crystal

Commit message: qwer
Parts:
- C1, C2: value C -> 12p; Mouser Part Number (none) -> C1206C120J5GACAUTO
- C3, C4, C5, C6, C7: Mouser Part Number (none) -> C1206X104J9RAL7210
- R1: Mouser Part Number (none) -> 1206W4J0102T5E
- R2: Mouser Part Number (none) -> 1206W4J0202T5E
- R27: Mouser Part Number (none) -> RN73R2BTTD5001B25
- U1: Mouser Part Number (none) -> 556-ATMEGA328PB-AN
- Y1: value Crystal -> 16M; footprint Crystal:Crystal_HC18-U_Vertical -> SamacSys_Parts:XRCGB16M000FXN14R0; Mouser Part Number (none) -> 81-XRCGB16M000FXN14R
Other:
- note added: "8pF load"
Changed lines of the file:
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@@
     (effects (font (size 1.27 1.27) (thickness 0.254) bold) (justify left bottom))
+  )
+  (text "8pF load" (at 111.76 17.78 0)
+    (effects (font (size 1.27 1.27)) (justify left bottom))
   )
   (text "Programming" (at 36.83 72.39 0)
@@
       (effects (font (size 1.27 1.27)) hide)
     )
+    (property "Mouser Part Number" "C1206X104J9RAL7210" (at 143.51 24.13 0)
+      (effects (font (size 1.27 1.27)) hide)
+    )
     (pin "1")
     (pin "2")
@@
       (effects (font (size 1.27 1.27)) hide)
     )
+    (property "Mouser Part Number" "C1206X104J9RAL7210" (at 181.61 24.13 0)
+      (effects (font (size 1.27 1.27)) hide)
+    )
     (pin "1")
     (pin "2")
@@
       (effects (font (size 1.27 1.27)))
     )
-    (property "Value" "Crystal" (at 105.41 19.05 0)
-      (effects (font (size 1.27 1.27)))
-    )
-    (property "Footprint" "Crystal:Crystal_HC18-U_Vertical" (at 105.41 24.13 0)
-      (effects (font (size 1.27 1.27)) hide)
-    )
-    (property "Datasheet" "~" (at 105.41 24.13 0)
+    (property "Value" "16M" (at 105.41 19.05 0)
+      (effects (font (size 1.27 1.27)))
+    )
+    (property "Footprint" "SamacSys_Parts:XRCGB16M000FXN14R0" (at 105.41 24.13 0)
+      (effects (font (size 1.27 1.27)) hide)
+    )
+    (property "Datasheet" "https://www.mouser.es/datasheet/2/281/p79e-806516.pdf" (at 105.41 24.13 0)
+      (effects (font (size 1.27 1.27)) hide)
+    )
+    (property "Mouser Part Number" "81-XRCGB16M000FXN14R" (at 105.41 24.13 0)
       (effects (font (size 1.27 1.27)) hide)
     )
@@
       (effects (font (size 1.27 1.27)) hide)
     )
+    (property "Mouser Part Number" "C1206X104J9RAL7210" (at 156.21 24.13 0)
+      (effects (font (size 1.27 1.27)) hide)
+    )
     (pin "1")
     (pin "2")
@@
     )
     (property "Datasheet" "~" (at 19.05 148.59 0)
+      (effects (font (size 1.27 1.27)) hide)
+    )
+    (property "Mouser Part Number" "1206W4J0202T5E" (at 19.05 148.59 0)
       (effects (font (size 1.27 1.27)) hide)
     )
@@
     )
     (property "Datasheet" "http://ww1.microchip.com/downloads/en/DeviceDoc/40001906C.pdf" (at 166.37 92.71 0)
+      (effects (font (size 1.27 1.27)) hide)
+    )
+    (property "Mouser Part Number" "556-ATMEGA328PB-AN" (at 166.37 92.71 0)
       (effects (font (size 1.27 1.27)) hide)
     )
@@
       (effects (font (size 1.27 1.27)) hide)
     )
-    (property "Campo4" "" (at 19.05 137.16 0)
+    (property "Mouser Part Number" "1206W4J0102T5E" (at 19.05 137.16 0)
       (effects (font (size 1.27 1.27)) hide)
     )
@@
       (effects (font (size 1.27 1.27)) hide)
     )
+    (property "Mouser Part Number" "C1206X104J9RAL7210" (at 168.91 24.13 0)
+      (effects (font (size 1.27 1.27)) hide)
+    )
     (pin "1")
     (pin "2")
@@
       (effects (font (size 1.27 1.27)) (justify right))
     )
-    (property "Value" "C" (at 115.57 33.02 0)
+    (property "Value" "12p" (at 115.57 33.02 0)
       (effects (font (size 1.27 1.27)) (justify right))
     )
@@
     )
     (property "Datasheet" "~" (at 111.76 31.75 0)
+      (effects (font (size 1.27 1.27)) hide)
+    )
+    (property "Mouser Part Number" "C1206C120J5GACAUTO" (at 111.76 31.75 0)
       (effects (font (size 1.27 1.27)) hide)
     )
@@
       (effects (font (size 1.27 1.27)) (justify right))
     )
-    (property "Value" "C" (at 101.6 33.02 0)
+    (property "Value" "12p" (at 101.6 33.02 0)
       (effects (font (size 1.27 1.27)) (justify right))
     )
@@
     )
     (property "Datasheet" "~" (at 97.79 31.75 0)
+      (effects (font (size 1.27 1.27)) hide)
+    )
+    (property "Mouser Part Number" "C1206C120J5GACAUTO" (at 97.79 31.75 0)
       (effects (font (size 1.27 1.27)) hide)
     )
@@
     )
     (property "Datasheet" "~" (at 194.31 24.13 0)
+      (effects (font (size 1.27 1.27)) hide)
+    )
+    (property "Mouser Part Number" "C1206X104J9RAL7210" (at 194.31 24.13 0)
       (effects (font (size 1.27 1.27)) hide)
     )
@@
       (effects (font (size 1.27 1.27)) hide)
     )
+    (property "Mouser Part Number" "RN73R2BTTD5001B25" (at 20.32 118.11 0)
+      (effects (font (size 1.27 1.27)) hide)
+    )

Commit message: BOM
Parts:
- removed Y1: 16M, SamacSys_Parts:XRCGB16M000FXN14R0, symbol Device:Crystal
- added Y2: 16M, SamacSys_Parts:ECS1601036CKMTR3, symbol Device:Crystal_GND24
- C1, C2, C3, C4, C5, C6, C7: footprint Capacitor_SMD:C_1206_3216Metric_Pad1.33x1.80mm_HandSolder -> Capacitor_SMD:C_1206_3216Metric
- R1, R2, R26, R27, R7: footprint Resistor_SMD:R_1206_3216Metric_Pad1.30x1.75mm_HandSolder -> Resistor_SMD:R_1206_3216Metric
Connections:
- net Earth: now also Y2.2, Y2.4
- net XTAL1: now also Y2.3
- net XTAL2: now also Y2.1
Other:
- note added: "10pF load"
- note removed: "8pF load"
Changed lines of the file:
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@@
+    (stroke (width 0) (type default))
+  )
+  (wire (pts (xy 105.41 29.21) (xy 105.41 35.56))
     (stroke (width 0) (type default))
   )
@@
     (effects (font (size 1.27 1.27) (thickness 0.254) bold) (justify left bottom))
   )
-  (text "8pF load" (at 111.76 17.78 0)
+  (text "10pF load" (at 111.76 17.78 0)
     (effects (font (size 1.27 1.27)) (justify left bottom))
   )
@@
       (effects (font (size 1.27 1.27)) (justify right))
     )
-    (property "Footprint" "Capacitor_SMD:C_1206_3216Metric_Pad1.33x1.80mm_HandSolder" (at 142.5448 20.32 0)
+    (property "Footprint" "Capacitor_SMD:C_1206_3216Metric" (at 142.5448 20.32 0)
       (effects (font (size 1.27 1.27)) hide)
     )
@@
       (effects (font (size 1.27 1.27)) (justify right))
     )
-    (property "Footprint" "Capacitor_SMD:C_1206_3216Metric_Pad1.33x1.80mm_HandSolder" (at 180.6448 20.32 0)
+    (property "Footprint" "Capacitor_SMD:C_1206_3216Metric" (at 180.6448 20.32 0)
       (effects (font (size 1.27 1.27)) hide)
     )
@@
     )
   )
+  (symbol (lib_id "power:Earth") (at 105.41 19.05 180) (unit 1)
+    (in_bom yes) (on_board yes) (dnp no) (fields_autoplaced)
+    (property "Reference" "#PWR0122" (at 105.41 12.7 0)
+      (effects (font (size 1.27 1.27)) hide)
+    )
+    (property "Value" "Earth" (at 105.41 15.24 0)
+      (effects (font (size 1.27 1.27)) hide)
+    )
+    (property "Footprint" "" (at 105.41 19.05 0)
+      (effects (font (size 1.27 1.27)) hide)
+    )
+    (property "Datasheet" "~" (at 105.41 19.05 0)
+      (effects (font (size 1.27 1.27)) hide)
+    )
+    (pin "1")
+    (instances
+      (project "KiCad"
+        (path "/557850ac-a946-4dff-8187-8978353577df"
+          (reference "#PWR0122") (unit 1)
+        )
+      )
+      (project "SalveNode"
+        (path "/947c7390-073c-40c7-ae18-83309c4a488f"
+          (reference "#PWR017") (unit 1)
+        )
+      )
+    )
+  )
   (symbol (lib_name "+5V_1") (lib_id "power:+5V") (at 19.05 133.35 0) (unit 1)
     (in_bom yes) (on_board yes) (dnp no) (fields_autoplaced)
@@
         (path "/947c7390-073c-40c7-ae18-83309c4a488f"
           (reference "#PWR01") (unit 1)
-        )
-      )
-    )
-  )
-  (symbol (lib_id "Device:Crystal") (at 105.41 24.13 0) (unit 1)
-    (in_bom yes) (on_board yes) (dnp no) (fields_autoplaced)
-    (property "Reference" "Y1" (at 105.41 16.51 0)
-      (effects (font (size 1.27 1.27)))
-    )
-    (property "Value" "16M" (at 105.41 19.05 0)
-      (effects (font (size 1.27 1.27)))
-    )
-    (property "Footprint" "SamacSys_Parts:XRCGB16M000FXN14R0" (at 105.41 24.13 0)
-      (effects (font (size 1.27 1.27)) hide)
-    )
-    (property "Datasheet" "https://www.mouser.es/datasheet/2/281/p79e-806516.pdf" (at 105.41 24.13 0)
-      (effects (font (size 1.27 1.27)) hide)
-    )
-    (property "Mouser Part Number" "81-XRCGB16M000FXN14R" (at 105.41 24.13 0)
-      (effects (font (size 1.27 1.27)) hide)
-    )
-    (pin "1")
-    (pin "2")
-    (instances
-      (project "SalveNode"
-        (path "/947c7390-073c-40c7-ae18-83309c4a488f"
-          (reference "Y1") (unit 1)
         )
       )
@@
         (path "/947c7390-073c-40c7-ae18-83309c4a488f"
           (reference "#PWR04") (unit 1)
+        )
+      )
+    )
+  )
+  (symbol (lib_id "Device:Crystal_GND24") (at 105.41 24.13 0) (unit 1)
+    (in_bom yes) (on_board yes) (dnp no)
+    (property "Reference" "Y2" (at 109.22 19.05 0)
+      (effects (font (size 1.27 1.27)))
+    )
+    (property "Value" "16M" (at 100.33 19.05 0)
+      (effects (font (size 1.27 1.27)))
+    )
+    (property "Footprint" "SamacSys_Parts:ECS1601036CKMTR3" (at 105.41 24.13 0)
+      (effects (font (size 1.27 1.27)) hide)
+    )
+    (property "Datasheet" "https://www.mouser.es/datasheet/2/281/p79e-806516.pdf" (at 105.41 24.13 0)
+      (effects (font (size 1.27 1.27)) hide)
+    )
+    (property "Mouser Part Number" "81-XRCGB16M000FXN14R" (at 105.41 24.13 0)
+      (effects (font (size 1.27 1.27)) hide)
+    )
+    (pin "1")
+    (pin "2")
+    (pin "3")
+    (pin "4")
+    (instances
+      (project "SalveNode"
+        (path "/947c7390-073c-40c7-ae18-83309c4a488f"
+          (reference "Y2") (unit 1)
         )
       )
@@
       (effects (font (size 1.27 1.27)) (justify right))
     )
-    (property "Footprint" "Capacitor_SMD:C_1206_3216Metric_Pad1.33x1.80mm_HandSolder" (at 155.2448 20.32 0)
+    (property "Footprint" "Capacitor_SMD:C_1206_3216Metric" (at 155.2448 20.32 0)
       (effects (font (size 1.27 1.27)) hide)
     )
@@
       (effects (font (size 1.27 1.27)) (justify left))
     )
-    (property "Footprint" "Resistor_SMD:R_1206_3216Metric_Pad1.30x1.75mm_HandSolder" (at 126.492 91.44 90)
+    (property "Footprint" "Resistor_SMD:R_1206_3216Metric" (at 126.492 91.44 90)
       (effects (font (size 1.27 1.27)) hide)
     )
@@
       (effects (font (size 1.27 1.27)) (justify left))
     )
-    (property "Footprint" "Resistor_SMD:R_1206_3216Metric_Pad1.30x1.75mm_HandSolder" (at 126.492 101.6 90)
+    (property "Footprint" "Resistor_SMD:R_1206_3216Metric" (at 126.492 101.6 90)
       (effects (font (size 1.27 1.27)) hide)
     )
@@
       (effects (font (size 1.27 1.27)) (justify left))
     )
-    (property "Footprint" "Resistor_SMD:R_1206_3216Metric_Pad1.30x1.75mm_HandSolder" (at 17.272 148.59 90)
+    (property "Footprint" "Resistor_SMD:R_1206_3216Metric" (at 17.272 148.59 90)
       (effects (font (size 1.27 1.27)) hide)
     )
@@
       (effects (font (size 1.27 1.27)) (justify right))
     )
-    (property "Footprint" "Resistor_SMD:R_1206_3216Metric_Pad1.30x1.75mm_HandSolder" (at 64.008 55.88 90)
+    (property "Footprint" "Resistor_SMD:R_1206_3216Metric" (at 64.008 55.88 90)
       (effects (font (size 1.27 1.27)) hide)
     )
@@
       (effects (font (size 1.27 1.27)) (justify left))
     )
-    (property "Footprint" "Resistor_SMD:R_1206_3216Metric_Pad1.30x1.75mm_HandSolder" (at 17.272 137.16 90)
+    (property "Footprint" "Resistor_SMD:R_1206_3216Metric" (at 17.272 137.16 90)
       (effects (font (size 1.27 1.27)) hide)
     )
@@
       (effects (font (size 1.27 1.27)))
     )
-    (property "Footprint" "Resistor_SMD:R_1206_3216Metric_Pad1.30x1.75mm_HandSolder" (at 34.29 90.932 90)
+    (property "Footprint" "Resistor_SMD:R_1206_3216Metric" (at 34.29 90.932 90)
       (effects (font (size 1.27 1.27)) hide)
     )
@@
       (effects (font (size 1.27 1.27)) (justify right))
     )
-    (property "Footprint" "Capacitor_SMD:C_1206_3216Metric_Pad1.33x1.80mm_HandSolder" (at 167.9448 20.32 0)
+    (property "Footprint" "Capacitor_SMD:C_1206_3216Metric" (at 167.9448 20.32 0)
       (effects (font (size 1.27 1.27)) hide)
     )
@@
       (effects (font (size 1.27 1.27)) (justify right))
     )
-    (property "Footprint" "Capacitor_SMD:C_1206_3216Metric_Pad1.33x1.80mm_HandSolder" (at 110.7948 27.94 0)
+    (property "Footprint" "Capacitor_SMD:C_1206_3216Metric" (at 110.7948 27.94 0)
       (effects (font (size 1.27 1.27)) hide)
     )
@@
       (effects (font (size 1.27 1.27)) (justify right))
     )
-    (property "Footprint" "Capacitor_SMD:C_1206_3216Metric_Pad1.33x1.80mm_HandSolder" (at 96.8248 27.94 0)
+    (property "Footprint" "Capacitor_SMD:C_1206_3216Metric" (at 96.8248 27.94 0)
       (effects (font (size 1.27 1.27)) hide)
     )
@@
       (effects (font (size 1.27 1.27)) (justify right))
     )
-    (property "Footprint" "Capacitor_SMD:C_1206_3216Metric_Pad1.33x1.80mm_HandSolder" (at 193.3448 20.32 0)
+    (property "Footprint" "Capacitor_SMD:C_1206_3216Metric" (at 193.3448 20.32 0)
       (effects (font (size 1.27 1.27)) hide)
     )
@@
       (effects (font (size 1.27 1.27)) (justify left))
     )
-    (property "Footprint" "Resistor_SMD:R_1206_3216Metric_Pad1.30x1.75mm_HandSolder" (at 18.542 118.11 90)
-      (effects (font (size 1.27 1.27)) hide)
-    )
+    (property "Footprint" "Resistor_SMD:R_1206_3216Metric" (at 18.542 118.11 90)
+      (effects (font (size 1.27 1.27)) hide)
+    )

Commit message: BOMS
Parts:
- R1: Mouser Part Number 1206W4J0102T5E -> 279-CRGCQ1206F1K0
- R2: Mouser Part Number 1206W4J0202T5E -> 71-CRCW12062K00JNEAC
- R27: Mouser Part Number RN73R2BTTD5001B25 -> 660-RN73R2BTTD5001B2
Changed lines of the file:
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@@
       (effects (font (size 1.27 1.27)) hide)
     )
-    (property "Mouser Part Number" "1206W4J0202T5E" (at 19.05 148.59 0)
+    (property "Mouser Part Number" "71-CRCW12062K00JNEAC" (at 19.05 148.59 0)
       (effects (font (size 1.27 1.27)) hide)
     )
@@
       (effects (font (size 1.27 1.27)) hide)
     )
-    (property "Mouser Part Number" "1206W4J0102T5E" (at 19.05 137.16 0)
+    (property "Mouser Part Number" "279-CRGCQ1206F1K0" (at 19.05 137.16 0)
       (effects (font (size 1.27 1.27)) hide)
     )
@@
       (effects (font (size 1.27 1.27)) hide)
     )
-    (property "Mouser Part Number" "RN73R2BTTD5001B25" (at 20.32 118.11 0)
-      (effects (font (size 1.27 1.27)) hide)
-    )
+    (property "Mouser Part Number" "660-RN73R2BTTD5001B2" (at 20.32 118.11 0)
+      (effects (font (size 1.27 1.27)) hide)
+    )

Commit message: BOM and PCB updated
Parts:
- removed J1, J21: Screw_Terminal_01x06, TerminalBlock_Phoenix:TerminalBlock_Phoenix_MKDS-1,5-6_1x06_P5.00mm_Horizontal, symbol Connector:Screw_Terminal_01x06
- added J2: AVR-ISP-6, Connector_PinHeader_1.00mm:PinHeader_2x03_P1.00mm_Vertical, symbol Connector:AVR-ISP-6
- added J3: 691382040006, SimbolosSnapEDA:691382040006, symbol 691382040006:691382040006
- R7: value PAD -> 10k; Mouser Part Number (none) -> 603-RT1206FRE1310KL
Connections:
- net +5V: now also J2.2 (VCC), J3.1
- net D0+: now also J3.3
- net D0-: now also J3.2
- net Earth: now also J2.6 (GND), J3.6
- net MISO: now also J2.1 (MISO)
- net MOSI: now also J2.4 (MOSI)
- net RESET: now also J2.5 (~{RST})
- net RI+: now also J3.5
- net RI-: now also J3.4
- net SCK: now also J2.3 (SCK)
Other:
- moved on the sheet: IC2, IC3, R1, R2, R27, R7

Commit message: fixes 2
Parts:
- removed R1: 1k, Resistor_SMD:R_1206_3216Metric, symbol Device:R
- removed R2: 2k, Resistor_SMD:R_1206_3216Metric, symbol Device:R
- added C1, C9: 1u, Capacitor_SMD:C_1206_3216Metric, symbol Device:C
- added U1: MCP1700x-330xxTT, Package_TO_SOT_SMD:SOT-23, symbol Regulator_Linear:MCP1700x-330xxTT
- R26, R27: value PAD -> 4.7k; Mouser Part Number (none) -> 603-RT1206FRE074K7L
- renumbered C1 to C2, C2 to C3, C3 to C4, C4 to C5, C5 to C6, C6 to C7, C7 to C8, J2 to J1, J3 to J2, U1 to U2, Y2 to Y1
Connections:
- net +5V: now also C1.2, U1.3 (VI)
- net Earth: now also C1.1, C9.1, U1.1 (GND)
- net +3.3V: now reaches IC3.2 (VDD)
- net +3.3V: now also C9.2, U1.2 (VO)
Other:
- moved on the sheet: IC3
