File: KiCad/IrrigationController/KiCad.kicad_sch (KiCad schematic)
At the start: 121 parts, among them IC1 MCP23017-E_SO, IC2 MCP23017-E_SO, IC3 DS89C21TMX_NOPB, J1 Screw_Terminal_01x03, J10 Screw_Terminal_01x05, J11 Screw_Terminal_01x02, J12 Screw_Terminal_01x02, J13 Screw_Terminal_01x04, J14 Screw_Terminal_01x02, J15 Screw_Terminal_01x02, J16 Screw_Terminal_01x02, J17 Screw_Terminal_01x02, J18 Screw_Terminal_01x02, J19 Screw_Terminal_01x02, J2 Screw_Terminal_01x03, J20 Screw_Terminal_01x05, J3 Screw_Terminal_01x03, J4 Screw_Terminal_01x03, J5 Screw_Terminal_01x03, J6 Screw_Terminal_01x02, J7 Screw_Terminal_01x02, J8 Screw_Terminal_01x02, J9 Screw_Terminal_01x02, K1 2071556-9, K2 2071556-9, Q1 2N3906, Q11 2N3904, Q12 2N3904, Q2 2N3906, Q3 2N3906, Q4 2N3906, Q6 2N3904, Q7 2N3904, Q8 2N3904, Q9 2N3904, SW1 SW_Push, U1 L298HN, U2 ARDUINO_MKR_WAN_1310, U3 L298HN, U4 L298HN, U5 L298HN, U7 L7805

Commit message: added other sch
Parts:
- removed D7, D8: 1N5711UR, Diode_SMD:D_1206_3216Metric_Pad1.42x1.75mm_HandSolder, symbol Diode:1N5711UR
- removed J4: Screw_Terminal_01x03, TerminalBlock_Phoenix:TerminalBlock_Phoenix_MKDS-1,5-3_1x03_P5.00mm_Horizontal, symbol Connector:Screw_Terminal_01x03
- removed Q4: 2N3906, Package_TO_SOT_SMD:SOT-23, symbol Transistor_BJT:2N3906
- removed Q9: 2N3904, Package_TO_SOT_SMD:SOT-23, symbol Transistor_BJT:2N3904
- removed R14: 4.7k, Resistor_SMD:R_1206_3216Metric_Pad1.30x1.75mm_HandSolder, symbol Device:R
- removed R19: 10k, Resistor_SMD:R_1206_3216Metric_Pad1.30x1.75mm_HandSolder, symbol Device:R
- removed R24: 27k, Resistor_SMD:R_1206_3216Metric_Pad1.30x1.75mm_HandSolder, symbol Device:R
- removed R8: 3.3k, Resistor_SMD:R_1206_3216Metric_Pad1.30x1.75mm_HandSolder, symbol Device:R
- R7: value 1.7k -> PAD
Connections:
- net RI_1: now also R7.2
- net RI_2: now also R7.1
- net S_ILUM_IN: no longer R7.2
Other:
- moved on the sheet: C13, C14, D1, D11, D12, D13, D14, D15, D16, D17, D18, D19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

Commit message: fixed err
Connections:
- net +3V3 is gone; now on net +3.3V: D1.1 (K), D3.1 (K), D5.1 (K), R17.2, R18.2
- net +9V is gone; now on net +12V: J5.1 (Pin_1)
- net +12V: now also C14.1, J19.2 (Pin_2), U7.1 (IN)
- net S_ILUM_EN: no longer names the net of U2.J3_12 (PA11/D3(PWM))
- net S_ILUM_IN: no longer names the net of U2.J3_5 (PA04/D18(PWM)/AIN(4)/A3)
- no-connect marks 21 -> 23
Other:
- moved on the sheet: C13, C14, J19, U7

Commit message: q
Changed lines of the file:
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@@
     (fill (type none))
   )
-  (text_box "Conector/Cable?"
-    (at 254 34.29 0) (size 60.96 30.48)
+  (text_box "METER UN PUNTO MAS PARA ALIMENTACION DE ESCALVO\n\nUSAR EL 328P DIRECTAMENTE"
+    (at 256.54 34.29 0) (size 43.18 34.29)
     (stroke (width 0) (type default))
     (fill (type none))

Commit message: tarjeta externa añadido
Parts:
- removed J20: Screw_Terminal_01x05, TerminalBlock_Phoenix:TerminalBlock_Phoenix_MKDS-1,5-5_1x05_P5.00mm_Horizontal, symbol Connector:Screw_Terminal_01x05
- added J21: Screw_Terminal_01x06, symbol Connector:Screw_Terminal_01x06
Connections:
- net +5V: now also J21.1 (Pin_1)
- net D0_1: now also J21.2 (Pin_2)
- net D0_2: now also J21.3 (Pin_3)
- net Earth: now also J21.6 (Pin_6)
- net RI_1: now also J21.4 (Pin_4)
- net RI_2: now also J21.5 (Pin_5)
Other:
- moved on the sheet: C13, C14, J19, U7

Commit message: qwer
Parts:
- Q3: Ref Mouser (none) -> 637-2N3906
Changed lines of the file:
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@@
       (effects (font (size 1.27 1.27)) (justify left) hide)
+    )
+    (property "Ref Mouser" "637-2N3906" (at 31.75 143.51 0)
+      (effects (font (size 1.27 1.27)) hide)
     )
     (pin "1")

Commit message: BOMS
Parts:
- removed D1, D2, D3, D4, D5, D6: 1N5711UR, Diode_SMD:D_1206_3216Metric_Pad1.42x1.75mm_HandSolder, symbol Diode:1N5711UR
- added D1, D2, D7: BAT54S, Package_TO_SOT_SMD:SOT-23, symbol Diode:BAT54S
- C1, C10, C11, C12, C13, C2, C3, C4, C5, C6, C7, C8, C9: footprint Capacitor_SMD:C_1206_3216Metric_Pad1.33x1.80mm_HandSolder -> Capacitor_SMD:C_1206_3216Metric; Mouser Part Number (none) -> 80-C1206C104J4GAUTO
- C14: footprint Capacitor_SMD:C_1206_3216Metric_Pad1.33x1.80mm_HandSolder -> Capacitor_SMD:C_1206_3216Metric; Mouser Part Number (none) -> 80-C1206C334K1RECAUT
- D11, D12, D13, D14, D15, D16, D17, D18, D19, D20, D21, D22, D23, D24, D25, D26, D27, D28, D29, D30, D31, D32, D33, D34, D35, D36, D37, D38, D39, D40, D41, D42: value 1N4007 -> SS24; footprint Diode_SMD:D_1206_3216Metric_Pad1.42x1.75mm_HandSolder -> Diode_SMD:D_SMB; Mouser Part Number (none) -> 821-SS24
- J21: footprint (none) -> TerminalBlock_Phoenix:TerminalBlock_Phoenix_MKDS-1,5-6_1x06_P5.00mm_Horizontal
- Q1, Q2, Q3: value 2N3906 -> MMBT3906; Mouser Part Number (none) -> 637-MMBT3906
- Q11, Q12, Q6, Q7, Q8: value 2N3904 -> MMBT3904; Mouser Part Number (none) -> 637-MMBT3904-AQ
- R1, R3, R5: value 1.7k -> 1.8k; footprint Resistor_SMD:R_1206_3216Metric_Pad1.30x1.75mm_HandSolder -> Resistor_SMD:R_1206_3216Metric; Mouser Part Number (none) -> 603-RT1206FRE071K8L
- R11, R12, R13: footprint Resistor_SMD:R_1206_3216Metric_Pad1.30x1.75mm_HandSolder -> Resistor_SMD:R_1206_3216Metric; Mouser Part Number (none) -> 603-RT1206FRE074K7L
- R16, R17, R18, R28: footprint Resistor_SMD:R_1206_3216Metric_Pad1.30x1.75mm_HandSolder -> Resistor_SMD:R_1206_3216Metric; Mouser Part Number (none) -> 603-RT1206FRE1310KL
- R2, R4, R6: footprint Resistor_SMD:R_1206_3216Metric_Pad1.30x1.75mm_HandSolder -> Resistor_SMD:R_1206_3216Metric; Mouser Part Number (none) -> 603-RT1206FRE073K3L
- R21, R22, R23: footprint Resistor_SMD:R_1206_3216Metric_Pad1.30x1.75mm_HandSolder -> Resistor_SMD:R_1206_3216Metric; Mouser Part Number (none) -> 603-RT1206FRE0727KL
- R26, R27, R7: footprint Resistor_SMD:R_1206_3216Metric_Pad1.30x1.75mm_HandSolder -> Resistor_SMD:R_1206_3216Metric
- R29, R30: footprint Resistor_SMD:R_1206_3216Metric_Pad1.30x1.75mm_HandSolder -> Resistor_SMD:R_1206_3216Metric; Mouser Part Number (none) -> 603-RT1206FRE071K5L
- U1, U3, U4, U5: value L298HN -> L298P; Mouser Part Number (none) -> 511-L298P
- U7: footprint Package_TO_SOT_THT:TO-220-3_Vertical -> Package_TO_SOT_SMD:TO-263-2; Mouser Part Number (none) -> 511-L7805ABD2T-TR
Connections:
- net +3.3V: now also D1.2 (K), D2.2 (K), D7.2 (K)
- net Earth: now also D1.1 (A), D2.1 (A), D7.1 (A)
- net S_HUM_1_IN: now also D7.3 (COM)
- net S_HUM_2_IN: now also D1.3 (COM)
- net S_HUM_3_IN: now also D2.3 (COM)

Commit message: qwer
Parts:
- added TP1, TP2: TestPoint, symbol Connector:TestPoint
- IC3: footprint SOIC127P600X175-8N -> SamacSys_Parts:SOP65P490X110-8N
Connections:
- net RX: now also TP2.1
- net TX: now also TP1.1
Changed lines of the file:
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@@
     (stroke (width 0) (type default))
   )
+  (wire (pts (xy 379.73 102.87) (xy 379.73 107.95))
+    (stroke (width 0) (type default))
+  )
   (wire (pts (xy 243.84 184.15) (xy 243.84 185.42))
     (stroke (width 0) (type default))
@@
     (stroke (width 0) (type default))
   )
+  (wire (pts (xy 394.97 102.87) (xy 394.97 107.95))
+    (stroke (width 0) (type default))
+  )
   (wire (pts (xy 185.42 167.64) (xy 185.42 185.42))
     (stroke (width 0) (type default))
@@
     (effects (font (size 1.27 1.27)) (justify left bottom))
   )
+  (label "RX" (at 394.97 107.95 90) (fields_autoplaced)
+    (effects (font (size 1.27 1.27)) (justify left bottom))
+  )
   (label "R1_EN" (at 119.38 132.08 90) (fields_autoplaced)
     (effects (font (size 1.27 1.27)) (justify left bottom))
@@
     (effects (font (size 1.27 1.27)) (justify left bottom))
   )
+  (label "TX" (at 379.73 107.95 90) (fields_autoplaced)
+    (effects (font (size 1.27 1.27)) (justify left bottom))
+  )
   (label "P3_IN1" (at 26.67 257.81 180) (fields_autoplaced)
     (effects (font (size 1.27 1.27)) (justify right bottom))
@@
     )
   )
+  (symbol (lib_id "Connector:TestPoint") (at 379.73 102.87 0) (unit 1)
+    (in_bom yes) (on_board yes) (dnp no) (fields_autoplaced)
+    (property "Reference" "TP1" (at 382.27 98.298 0)
+      (effects (font (size 1.27 1.27)) (justify left))
+    )
+    (property "Value" "TestPoint" (at 382.27 100.838 0)
+      (effects (font (size 1.27 1.27)) (justify left))
+    )
+    (property "Footprint" "" (at 384.81 102.87 0)
+      (effects (font (size 1.27 1.27)) hide)
+    )
+    (property "Datasheet" "~" (at 384.81 102.87 0)
+      (effects (font (size 1.27 1.27)) hide)
+    )
+    (pin "1")
+    (instances
+      (project "KiCad"
+        (path "/557850ac-a946-4dff-8187-8978353577df"
+          (reference "TP1") (unit 1)
+        )
+      )
+    )
+  )
   (symbol (lib_id "Transistor_BJT:2N3904") (at 210.82 271.78 0) (unit 1)
     (in_bom yes) (on_board yes) (dnp no)
@@
     )
   )
+  (symbol (lib_id "Connector:TestPoint") (at 394.97 102.87 0) (unit 1)
+    (in_bom yes) (on_board yes) (dnp no) (fields_autoplaced)
+    (property "Reference" "TP2" (at 397.51 98.298 0)
+      (effects (font (size 1.27 1.27)) (justify left))
+    )
+    (property "Value" "TestPoint" (at 397.51 100.838 0)
+      (effects (font (size 1.27 1.27)) (justify left))
+    )
+    (property "Footprint" "" (at 400.05 102.87 0)
+      (effects (font (size 1.27 1.27)) hide)
+    )
+    (property "Datasheet" "~" (at 400.05 102.87 0)
+      (effects (font (size 1.27 1.27)) hide)
+    )
+    (pin "1")
+    (instances
+      (project "KiCad"
+        (path "/557850ac-a946-4dff-8187-8978353577df"
+          (reference "TP2") (unit 1)
+        )
+      )
+    )
+  )
   (symbol (lib_id "ARDUINO_MKR_WAN_1310:ARDUINO_MKR_WAN_1310") (at 158.75 46.99 0) (unit 1)
     (in_bom yes) (on_board yes) (dnp no) (fields_autoplaced)
@@
       (effects (font (size 1.27 1.27)))
     )
-    (property "Footprint" "SOIC127P600X175-8N" (at 260.35 365.43 0)
+    (property "Footprint" "SamacSys_Parts:SOP65P490X110-8N" (at 260.35 365.43 0)
       (effects (font (size 1.27 1.27)) (justify left top) hide)
     )

Commit message: qwer
Parts:
- removed U1, U3, U4, U5: L298P, Package_TO_SOT_THT:TO-220-15_P2.54x2.54mm_StaggerOdd_Lead4.58mm_Vertical, symbol Driver_Motor:L298HN
- added C15, C16, C17, C18: 100n, Capacitor_SMD:C_1206_3216Metric, symbol Device:C
- added U1, U3, U4, U5: L298P, Package_SO:HSOP-20-1EP_11.0x15.9mm_P1.27mm_SlugDown_ThermalVias, symbol Driver_Motor:L298P
- TP1, TP2: footprint (none) -> TestPoint:TestPoint_Pad_2.0x2.0mm
Connections:
- net +12V: now also U1.6 (Vs), U3.6 (Vs), U4.6 (Vs), U5.6 (Vs)
- net +5V: now also C16.1, C17.1, C18.1, U1.12 (Vss), U3.12 (Vss), U4.12 (Vss), U5.12 (Vss)
- net Earth: now also C15.1, C16.2, C17.2, C18.2, U1.1 (GND), U1.10 (GND), U1.11 (GND), U1.19 (SENSE_B), U1.2 (SENSE_A), U1.20 (GND), U3.1 (GND), U3.10 (GND), U3.11 (GND), U3.19 (SENSE_B), U3.2 (SENSE_A), U3.20 (GND), U4.1 (GND), U4.10 (GND), U4.11 (GND), U4.19 (SENSE_B), U4.2 (SENSE_A), U4.20 (GND), U5.1 (GND), U5.10 (GND), U5.11 (GND), U5.19 (SENSE_B), U5.2 (SENSE_A), U5.20 (GND)
- net P1_EN: now also U5.8 (EnA)
- net P1_IN1: now also U5.9 (IN2)
- net P1_IN2: now also U5.7 (IN1)
- net P2_EN: now also U5.14 (EnB)
- net P2_IN1: now also U5.15 (IN4)
- net P2_IN2: now also U5.13 (IN3)
- net P3_EN: now also U4.8 (EnA)
- net P3_IN1: now also U4.9 (IN2)
- net P3_IN2: now also U4.7 (IN1)
- net P4_EN: now also U4.14 (EnB)
- net P4_IN1: now also U4.15 (IN4)
- net P4_IN2: now also U4.13 (IN3)
- net P5_EN: now also U3.8 (EnA)
- net P5_IN1: now also U3.9 (IN2)
- net P5_IN2: now also U3.7 (IN1)
- net R1_EN: now also U1.14 (EnB)
- net R1_IN1: now also U1.15 (IN4)
- net R1_IN2: now also U1.13 (IN3)
- net Vin: now also C15.2
- net W1_EN: now also U3.14 (EnB)
- net W1_IN1: now also U3.15 (IN4)
- net W1_IN2: now also U3.13 (IN3)
- net W2_EN: now also U1.8 (EnA)
- net W2_IN1: now also U1.9 (IN2)
- net W2_IN2: now also U1.7 (IN1)
- net at D29.2 (A), D30.1 (K), J11.1 (Pin_1): now also U4.16 (OUT3)
- net at D17.2 (A), D18.1 (K), J7.1 (Pin_1): now also U1.4 (OUT1)
- net at D15.2 (A), D16.1 (K), J7.2 (Pin_2): now also U1.5 (OUT2)
- net at D37.2 (A), D38.1 (K), J17.1 (Pin_1): now also U5.16 (OUT3)
- net at D19.2 (A), D20.1 (K), J8.2 (Pin_2): now also U3.17 (OUT4)
- net at D21.2 (A), D22.1 (K), J8.1 (Pin_1): now also U3.16 (OUT3)
- net at D41.2 (A), D42.1 (K), J18.1 (Pin_1): now also U5.4 (OUT1)
- net at D13.2 (A), D14.1 (K), J6.1 (Pin_1): now also U1.16 (OUT3)
- net at D39.2 (A), D40.1 (K), J18.2 (Pin_2): now also U5.5 (OUT2)
- net at D35.2 (A), D36.1 (K), J17.2 (Pin_2): now also U5.17 (OUT4)
- net at D27.2 (A), D28.1 (K), J11.2 (Pin_2): now also U4.17 (OUT4)
- net at D25.2 (A), D26.1 (K), J9.1 (Pin_1): now also U3.4 (OUT1)
- net at D23.2 (A), D24.1 (K), J9.2 (Pin_2): now also U3.5 (OUT2)
- net at D31.2 (A), D32.1 (K), J14.2 (Pin_2): now also U4.5 (OUT2)
- net at D33.2 (A), D34.1 (K), J14.1 (Pin_1): now also U4.4 (OUT1)
- net at D11.2 (A), D12.1 (K), J6.2 (Pin_2): now also U1.17 (OUT4)
- net D0_1 renamed D0+
- net D0_2 renamed D0-
- net RI_1 renamed RI+
- net RI_2 renamed RI-
