File: KiCad/IrrigationController/KiCad.kicad_pcb (KiCad board)
At the start: 2 copper layers, 121.5 x 115 mm, 113 parts, among them IC1 MCP23017-E_SO, IC2 MCP23017-E_SO, IC3 DS89C21TMX_NOPB, J1 Screw_Terminal_01x03, J10 Screw_Terminal_01x05, J11 Screw_Terminal_01x02, J12 Screw_Terminal_01x02, J13 Screw_Terminal_01x04, J14 Screw_Terminal_01x02, J15 Screw_Terminal_01x02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

Commit message: qwer
Routing:
- net /PULSE_IN: track 9.56 -> 80.6 mm, vias 0 -> 2
- net +5V: track 88.1 -> 78.5 mm, vias 11 -> 9
